File: Faston_and_Sun_LED-PCB.kicad_pcb (KiCad board)
At the start: 2 copper layers, 60 x 23 mm, 7 parts, among them J1 Barrel_Jack_Switch, J2 Conn_01x02_Female, J3 62409-1, J4 62409-1, U1 NSI45060JDT4G

Commit message: add V1.0.1 and output gerber
add V1.0.1 and output gerber
Parts:
- added J5: 63067-1_VCC, CRD_Sun_LED:63067-1, F.Cu at (114.8, 96.5)
- added J6: 63067-1_GND, CRD_Sun_LED:63067-1, F.Cu at (118.0, 103.0)
- added J7: 63969-1_VCC, CRD_Sun_LED:63969-1, F.Cu at (131.9, 96.5)
- added J8: 63969-1_GND, CRD_Sun_LED:63969-1, F.Cu at (135.0, 103.3)
- J3, J4: footprint BP5293_series:TE_62409-1 -> CRD_Sun_LED:TE_62409-1
- moved J1 5.71 mm to (127.5, 85.5)
- moved J2 5.71 mm to (135.4, 85.5)
- moved D1 1.91 mm to (164.0, 84.9)
- moved J3 1.91 mm to (149.0, 92.1)
- moved J4 1.91 mm to (148.5, 98.9)
- moved R1 1.91 mm to (160.6, 97.6)
- moved U1 1.91 mm to (168.5, 97.4)
Routing:
- net Net-(J1-Pad1): track 7.97 -> 49.7 mm
- net Net-(J1-Pad2): track 17.8 -> 54.1 mm
Other:
- board size 60 x 23 mm -> 60 x 28 mm
