File: Faston_and_Sun_LED-PCB.sch (KiCad schematic (older format))
At the start: 7 parts, among them J1 Barrel_Jack_Switch, J2 Conn_01x02_Female, J3 62409-1, J4 62409-1, U1 NSI45060JDT4G

Commit message: add pcb v1.0.0
add pcb v1.0.0
Parts:
- D1: footprint (none) -> CRD_Sun_LED:ENB01-NHSD7-F1
- J1: footprint (none) -> Connector_BarrelJack:BarrelJack_Horizontal
- J2: footprint (none) -> Connector_PinHeader_2.54mm:PinHeader_1x02_P2.54mm_Vertical
- R1: footprint (none) -> Resistor_THT:R_Axial_DIN0207_L6.3mm_D2.5mm_P2.54mm_Vertical
Changed lines of the file:
@@
 encoding utf-8
 Sheet 1 1
-Title ""
-Date ""
-Rev ""
-Comp ""
-Comment1 ""
+Title "Faston terminal and Blink Sun right like LED"
+Date "2020-11-29"
+Rev "V1.0.0"
+Comp "Geekhouse Tsukuba's Tomori Nao"
+Comment1 "Presented by takurx"
 Comment2 ""
 Comment3 ""
@@
 F 0 "J1" H 3557 3017 50  0000 C CNN
 F 1 "Barrel_Jack_Switch" H 3557 2926 50  0000 C CNN
-F 2 "" H 3550 2660 50  0001 C CNN
+F 2 "Connector_BarrelJack:BarrelJack_Horizontal" H 3550 2660 50  0001 C CNN
 F 3 "~" H 3550 2660 50  0001 C CNN
 	1    3500 2700
@@
 F 0 "D1" V 7139 2132 50  0000 R CNN
 F 1 "LED" V 7048 2132 50  0000 R CNN
-F 2 "" H 7100 2250 50  0001 C CNN
+F 2 "CRD_Sun_LED:ENB01-NHSD7-F1" H 7100 2250 50  0001 C CNN
 F 3 "~" H 7100 2250 50  0001 C CNN
 	1    7100 2250
@@
 F 0 "J2" H 4478 2576 50  0000 L CNN
 F 1 "Conn_01x02_Female" H 4478 2485 50  0000 L CNN
-F 2 "" H 4450 2600 50  0001 C CNN
+F 2 "Connector_PinHeader_2.54mm:PinHeader_1x02_P2.54mm_Vertical" H 4450 2600 50  0001 C CNN
 F 3 "~" H 4450 2600 50  0001 C CNN
 	1    4450 2600
@@
 F 0 "R1" H 7770 3596 50  0000 L CNN
 F 1 "R" H 7770 3505 50  0000 L CNN
-F 2 "" V 7630 3550 50  0001 C CNN
+F 2 "Resistor_THT:R_Axial_DIN0207_L6.3mm_D2.5mm_P2.54mm_Vertical" V 7630 3550 50  0001 C CNN
 F 3 "~" H 7700 3550 50  0001 C CNN
 	1    7700 3550
@@
 $EndComp
 Wire Wire Line
-	4250 2600 3800 2600
-Wire Wire Line
 	3800 2800 3950 2800
 Wire Wire Line
@@
 	3950 2700 3950 2800
 Connection ~ 3950 2800
-Wire Wire Line
-	3950 2800 4250 2800
 Wire Wire Line
 	7100 2100 6650 2100
@@
 	7700 3700 7100 3700
 Connection ~ 7100 3700
+Wire Wire Line
+	3950 2800 4250 2800
+Wire Wire Line
+	3800 2600 4250 2600
 $EndSCHEMATC

Commit message: add V1.0.1 and output gerber
add V1.0.1 and output gerber
Parts:
- added J5: 63067-1_VCC, CRD_Sun_LED:63067-1, symbol Connector:Conn_01x01_Male
- added J6: 63067-1_GND, CRD_Sun_LED:63067-1, symbol Connector:Conn_01x01_Male
- added J7: 63969-1_VCC, CRD_Sun_LED:63969-1, symbol Connector:Conn_01x01_Female
- added J8: 63969-1_GND, CRD_Sun_LED:63969-1, symbol Connector:Conn_01x01_Female
- J3, J4: footprint TE_62409-1 -> CRD_Sun_LED:TE_62409-1
Connections:
- net at J1.1, J2.1 (Pin_1): now also J5.1 (Pin_1), J7.1 (Pin_1)
- net at J1.2, J1.3, J2.2 (Pin_2): now also J6.1 (Pin_1), J8.1 (Pin_1)
Changed lines of the file:
@@
 F 0 "J3" H 5443 2283 50  0000 C CNN
 F 1 "62409-1" H 5443 2374 50  0000 C CNN
-F 2 "TE_62409-1" H 5550 2650 50  0001 L BNN
+F 2 "CRD_Sun_LED:TE_62409-1" H 5550 2650 50  0001 L BNN
 F 3 "" H 5550 2650 50  0001 L BNN
 F 4 "62409-1" H 5550 2650 50  0001 L BNN "Comment"
@@
 F 0 "J4" H 5443 2933 50  0000 C CNN
 F 1 "62409-1" H 5443 3024 50  0000 C CNN
-F 2 "TE_62409-1" H 5550 3300 50  0001 L BNN
+F 2 "CRD_Sun_LED:TE_62409-1" H 5550 3300 50  0001 L BNN
 F 3 "" H 5550 3300 50  0001 L BNN
 F 4 "62409-1" H 5550 3300 50  0001 L BNN "Comment"
@@
 	3950 2800 4250 2800
 Wire Wire Line
-	3800 2600 4250 2600
+	3800 2600 4100 2600
+$Comp
+L Connector:Conn_01x01_Male J6
+U 1 1 5FC458FE
+P 3800 3400
+F 0 "J6" V 3862 3444 50  0000 L CNN
+F 1 "63067-1_GND" H 3500 3300 50  0000 L CNN
+F 2 "CRD_Sun_LED:63067-1" H 3800 3400 50  0001 C CNN
+F 3 "~" H 3800 3400 50  0001 C CNN
+	1    3800 3400
+	0    -1   -1   0
+$EndComp
+$Comp
+L Connector:Conn_01x01_Male J5
+U 1 1 5FC4643C
+P 3550 3400
+F 0 "J5" V 3704 3312 50  0000 R CNN
+F 1 "63067-1_VCC" H 3750 3550 50  0000 R CNN
+F 2 "CRD_Sun_LED:63067-1" H 3550 3400 50  0001 C CNN
+F 3 "~" H 3550 3400 50  0001 C CNN
+	1    3550 3400
+	0    -1   -1   0
+$EndComp
+$Comp
+L Connector:Conn_01x01_Female J7
+U 1 1 5FC47A59
+P 4400 3400
+F 0 "J7" V 4246 3448 50  0000 L CNN
+F 1 "63969-1_VCC" H 4100 3200 50  0000 L CNN
+F 2 "CRD_Sun_LED:63969-1" H 4400 3400 50  0001 C CNN
+F 3 "~" H 4400 3400 50  0001 C CNN
+	1    4400 3400
+	0    1    1    0
+$EndComp
+$Comp
+L Connector:Conn_01x01_Female J8
+U 1 1 5FC4896F
+P 4650 3400
+F 0 "J8" V 4496 3448 50  0000 L CNN
+F 1 "63969-1_GND" H 4400 3600 50  0000 L CNN
+F 2 "CRD_Sun_LED:63969-1" H 4650 3400 50  0001 C CNN
+F 3 "~" H 4650 3400 50  0001 C CNN
+	1    4650 3400
+	0    1    1    0
+$EndComp
+Wire Wire Line
+	4650 3200 4650 2950
+Wire Wire Line
+	4650 2950 3950 2950
+Wire Wire Line
+	3950 2950 3950 2800
+Wire Wire Line
+	3950 2950 3800 2950
+Wire Wire Line
+	3800 2950 3800 3200
+Connection ~ 3950 2950
+Wire Wire Line
+	4400 3200 4400 3050
+Wire Wire Line
+	4400 3050 4100 3050
+Wire Wire Line
+	4100 3050 4100 2600
+Connection ~ 4100 2600
+Wire Wire Line
+	4100 2600 4250 2600
+Wire Wire Line
+	4100 3050 3550 3050
+Wire Wire Line
+	3550 3050 3550 3200
+Connection ~ 4100 3050
 $EndSCHEMATC
